File: Launch-Controller/launchController/launchController_noTemp.kicad_sch (KiCad schematic)
At the start: 103 parts, among them J1 Conn_01x05_Pin, J10 Conn_01x05_Pin, J11 Raspberry_Pi_5, J13 26 pin Dsub, J14 DB25_Plug, J16 DB25_Plug, J17 DB25_Plug, J2 Conn_01x05_Pin, J3 Conn_01x05_Pin, J4 Conn_01x05_Pin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

Commit message: dimensions
Parts:
- C10, C11, C12, C13, C14, C2, C3, C4, C5, C6, C7, C8, C9: footprint Capacitor_THT:C_Disc_D5.1mm_W3.2mm_P5.00mm -> Capacitor_SMD:C_0402_1005Metric_Pad0.74x0.62mm_HandSolder
- D1, D13, D14, D15, D16, D17, D18, D19, D20, D21, D22: footprint LED_THT:LED_D4.0mm -> LED_SMD:LED_1206_3216Metric_Pad1.42x1.75mm_HandSolder
- D10, D11, D12, D2, D3, D4, D5, D6, D7, D8, D9: footprint LED_THT:LED_D3.0mm -> LED_SMD:LED_0603_1608Metric_Pad1.05x0.95mm_HandSolder
- Q1, Q10, Q2, Q3, Q4, Q5, Q6, Q7, Q8, Q9: footprint Package_TO_SOT_THT:TO-220-3_Horizontal_TabDown -> Package_TO_SOT_SMD:SOT-23-3
- R1, R10, R11, R12, R3, R4, R5, R6, R7, R8, R9: footprint Resistor_THT:R_Axial_DIN0411_L9.9mm_D3.6mm_P12.70mm_Horizontal -> Resistor_SMD:R_0805_2012Metric_Pad1.20x1.40mm_HandSolder
- R13, R14, R15, R16, R17, R18, R19, R2, R20, R21, R22, R23, R24, R25, R26, R27, R28, R29, R30, R31, R32: footprint Resistor_THT:R_Axial_DIN0207_L6.3mm_D2.5mm_P7.62mm_Horizontal -> Resistor_SMD:R_1210_3225Metric_Pad1.30x2.65mm_HandSolder
- U1, U2: footprint SARP:ADS1015 -> launch_controller:ADS1115
