File: Launch-Controller/buck_converter/Buck5V2/Buck5.kicad_sch (KiCad schematic)
At the start: 10 parts, among them J1 Conn_01x10_Socket, U1 LM2596S-5

Commit message: buck converter mounting hole and dimension changes
Parts:
- added H1, H2: MountingHole_Pad, MountingHole:MountingHole_3.7mm_Pad, symbol Mechanical:MountingHole_Pad
Connections:
- net GND: now also H1.1, H2.1
Other:
- note added: "Buck Converter Circuit"
- note added: "Connector"
- note added: "Mounting Holes"
- moved on the sheet: Cin1, Cout1, D1, D2, D3, J1, L1, R1, R2, U1
