File: Launch-Controller/relays/RelaySwitchCompact.kicad_pcb (KiCad board)
At the start: 2 copper layers, 38.2 x 17 mm, 14 parts, among them J1 Conn_01x05_Pin, K1 1-1721150-0, U1 FOD817ASD, U2 FMMT634QTA

Commit message: finalized relay board
Other:
- board text added: "Owen Wilhere"
- board text added: "SARP"
