File: Launch-Controller/relays/RelaySwitchCompact.kicad_pcb (KiCad board)
At the start: 2 copper layers, 38.2 x 17 mm, 12 parts, among them J1 350-10-105-00-001101, K1 1-1721150-0, U1 FOD817ASD, U2 FMMT634QTA

Commit message: fab_files finalized
Parts:
- added F1: Fuse, Diode_SMD:D_0402_1005Metric_Pad0.77x0.64mm_HandSolder, B.Cu at (155.5, 97.7)
Connections:
- K1 pad 5: /RelayIn -> Net-(F1-Pad1)
Routing:
- net Net-(F1-Pad1): track 0.00 -> 3.60 mm
- net /RelayIn: track 6.77 -> 3.23 mm
